File: voltage_adjuster.kicad_sch (KiCad schematic)
At the start: 24 parts, among them IC1 LDK130PU-R, IC2 MCP73832T-2ACI_MC, J1 UJC-H-G-SMT-1-P6-TR

Commit message: fixed bom
Parts:
- C1, C2: Mouser Part Number 963-LMK107BJ475KA-T -> 963-LMK107BJ475KA-T
- C3, C4: Mouser Part Number 963-LMK107B7105KA-T -> 963-LMK107B7105KA-T
- D1: Mouser Part Number 859-LTST-C190KRKT -> 859-LTST-C190KRKT
- IC1: Manufacturer Part Number (none) -> LDK130PU-R; Mouser Part Number 511-LDK130PU-R -> 511-LDK130PU-R
- IC2: Manufacturer Part Number (none) -> MCP73832T-2ACI/MC; Mouser Part Number 579-MCP73832T-2ACIMC -> 579-MCP73832T-2ACIMC
- J1: Manufacturer Part Number (none) -> UJC-H-G-SMT-P6-TR; Mouser Part Number (none) -> 179-UJCHGSMTP6TR
- JP1, JP2, JP3, TP1, TP2, TP3, TP4, TP5: now left out of the parts list
- R1: Manufacturer Part Number CRG0603F56K -> CRG0603F56K; Mouser Part Number 279-CRG0603F56K -> 279-CRG0603F56K
- R2: Mouser Part Number 279-CRG0603F1K5 -> 279-CRG0603F1K5
- R5: Manufacturer Part Number CRG0603F56K -> RC0603FR-0788K7L; Mouser Part Number 279-CRG0603F56K -> 603-RC0603FR-0788K7L
- R6: Manufacturer Part Number CRG0603F56K -> RCA0603100KFKEC; Mouser Part Number 279-CRG0603F56K -> 71-RCA0603100KFKEC
- R7: Manufacturer Part Number CRG0603F56K -> AC0603FR-07124KL; Mouser Part Number 279-CRG0603F56K -> 603-AC0603FR-07124KL
- R8: Manufacturer Part Number CRG0603F56K -> AC0603FR-07316KL; Mouser Part Number 279-CRG0603F56K -> 603-AC0603FR-07316KL
